File: PCB/PCB.sch (KiCad schematic (older format))
At the start: 138 parts, among them SW1 SW_Push, U1 ATmega32U4-AU, Y1 16MHz

Commit message: Restarted work on key placement using new footprint.
Signed-off-by: Oscar <oscarwebb08@gmail.com>
Parts:
- MX1, MX10, MX11, MX12, MX13, MX14, MX15, MX16, MX18, MX19, MX20, MX21, MX23, MX24, MX25, MX26, MX28, MX29, MX30, MX31, MX33, MX34, MX35, MX36, MX38, MX39, MX40, MX41, MX43, MX44, MX45, MX46, MX48, MX49, MX5, MX50, MX51, MX53, MX54, MX55, MX57, MX58, MX6, MX7, MX8, MX9: footprint Kailh_Choc:KailhChoc-1U -> Switch_Keyboard_Kailh:SW_Kailh_Choc_V1_1.00u; symbol MX_Alps_Hybrid:MX-NoLED -> PCB-rescue:MX-NoLED-MX_Alps_Hybrid
- MX17, MX22, MX27, MX37, MX42, MX47, MX52: footprint Kailh_Choc:KailhChoc-1.25U -> Switch_Keyboard_Kailh:SW_Kailh_Choc_V1_1.25u; symbol MX_Alps_Hybrid:MX-NoLED -> PCB-rescue:MX-NoLED-MX_Alps_Hybrid
- MX2, MX61: footprint Kailh_Choc:KailhChoc-1U -> Switch_Keyboard_Kailh:SW_Kailh_Choc_V1_1.50u; symbol MX_Alps_Hybrid:MX-NoLED -> PCB-rescue:MX-NoLED-MX_Alps_Hybrid
- MX3: footprint Kailh_Choc:KailhChoc-1U -> Switch_Keyboard_Kailh:SW_Kailh_Choc_V1_1.75u; symbol MX_Alps_Hybrid:MX-NoLED -> PCB-rescue:MX-NoLED-MX_Alps_Hybrid
- MX32: footprint Kailh_Choc:KailhChoc-1.75U -> Switch_Keyboard_Kailh:SW_Kailh_Choc_V1_6.25u; symbol MX_Alps_Hybrid:MX-NoLED -> PCB-rescue:MX-NoLED-MX_Alps_Hybrid
- MX4, MX59: footprint Kailh_Choc:KailhChoc-1U -> Switch_Keyboard_Kailh:SW_Kailh_Choc_V1_2.25u; symbol MX_Alps_Hybrid:MX-NoLED -> PCB-rescue:MX-NoLED-MX_Alps_Hybrid
- MX56: footprint Kailh_Choc:KailhChoc-1U -> Switch_Keyboard_Kailh:SW_Kailh_Choc_V1_2.75u; symbol MX_Alps_Hybrid:MX-NoLED -> PCB-rescue:MX-NoLED-MX_Alps_Hybrid
- MX60: footprint Kailh_Choc:KailhChoc-1U -> Switch_Keyboard_Kailh:SW_Kailh_Choc_V1_2.00u; symbol MX_Alps_Hybrid:MX-NoLED -> PCB-rescue:MX-NoLED-MX_Alps_Hybrid
Connections:
- net 1: now also MX17.1 (COL)
- net 10: no longer MX47.1 (COL)
- net 11: now also MX37.1 (COL); no longer MX52.1 (COL)
- net 12: now also MX42.1 (COL)
- net 13: now also MX47.1 (COL)
- net 14: now also MX52.1 (COL)
- net 2: now also MX22.1 (COL)
- net 3: now also MX27.1 (COL)
- net 4: no longer MX17.1 (COL)
- net 5: no longer MX22.1 (COL)
- net 6: no longer MX27.1 (COL)
- net 8: no longer MX37.1 (COL)
- net 9: no longer MX42.1 (COL)
- net GND: no longer USB1.1 (GND)
- no-connect marks 2 -> 1
Other:
- moved on the sheet: D17, D22, D27, D37, D42, D47, D52, MX17, MX22, MX27, MX37, MX42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
